Commit message: Update to include ros controller

File: arctos/description/urdf/arctos.xacro (robot description, xacro)
@@ -1,7 +1,14 @@
 <?xml version="1.0" ?>
 <robot name="arctos" xmlns:xacro="http://www.ros.org/wiki/xacro">
-<xacro:include filename="$(find arctos_description)/urdf/materials.xacro" />
-<xacro:include filename="$(find arctos_description)/urdf/joint_link.xacro"/>
-<!--xacro:include filename="$(find arctos_description)/urdf/arctos_gripper.xacro"/-->
+<xacro:include filename="$(find arctos)/urdf/materials.xacro" />
+<xacro:include filename="$(find arctos)/urdf/joint_link.xacro"/>
+<link name="world"/>
+  <!-- base_joint fixes base_link to the environment -->
+  <joint name="base_joint" type="fixed">
+    <parent link="world"/>
+    <child link="base_link"/>
+    <origin xyz="0 0 0" rpy="0 0 0"/>
+    <axis xyz="0 0 1"/>
+  </joint>
 <xacro:arctos_link
     name="base_link"
@@ -56,9 +63,8 @@
     origin_xyz="0.0 0.323 -0.5685" origin_rpy="0 0 0"
     material_name="white"
-    inertia_origin_xyz="-0.001 -0.0211 0.0" inertia_origin_rpy="0 0 0"
-    mass="0.2858"
-    ixx="1e-4" iyy="1e-4" izz="1e-4" ixy="-0.0" iyz="0.0" ixz="0.0"
+    inertia_origin_xyz="-0.0 -0.0 0.0" inertia_origin_rpy="0.0 0.0 0.0"
+    mass="1e-3"
+    ixx="1e-3" iyy="1e-3" izz="1e-3" ixy="-0.0" iyz="0.0" ixz="0.0"
 />
-<!--xacro:gripper parent="Link_6_1" origin_xyz="0.0 -0.006085 0.0" /-->
 <xacro:arctos_joint
   name="X_joint" type="continuous"
@@ -103,9 +109,5 @@
   limit_u="${pi}" limit_l="${-pi}" limit_e="16.0" limit_v="3.0"
 />
-<xacro:transmission name="X_tran" joint_name="X_joint" actuator_name="X_actr"/>
-<xacro:transmission name="Y_tran" joint_name="Y_joint" actuator_name="Y_actr"/>
-<xacro:transmission name="B_tran" joint_name="B_joint" actuator_name="B_actr"/>
-<xacro:transmission name="Z_tran" joint_name="Z_joint" actuator_name="Z_actr"/>
-<xacro:transmission name="A_tran" joint_name="A_joint" actuator_name="A_actr"/>
-<xacro:transmission name="C_tran" joint_name="C_joint" actuator_name="C_actr"/>
+<!--xacro:include filename="$(find arctos)/urdf/arctos_gripper.xacro"/-->
+<xacro:include filename="$(find arctos)/urdf/arctos_control.xacro"/>
 </robot>

File: arctos/description/urdf/joint_link.xacro (robot description, xacro)
@@ -6,5 +6,5 @@
       <origin xyz="${origin_xyz}" rpy="${origin_rpy}"/>
       <geometry>
-        <mesh filename="package://arctos_description/meshes/${name}.stl" scale="0.001 0.001 0.001"/>
+        <mesh filename="package://arctos/meshes/${name}.stl" scale="0.001 0.001 0.001"/>
       </geometry>
       <material name="${material_name}"/>
@@ -13,5 +13,5 @@
       <origin xyz="${origin_xyz}" rpy="${origin_rpy}"/>
       <geometry>
-        <mesh filename="package://arctos_description/meshes/${name}.stl" scale="0.001 0.001 0.001"/>
+        <mesh filename="package://arctos/meshes/${name}.stl" scale="0.001 0.001 0.001"/>
       </geometry>
     </collision>
@@ -32,27 +32,13 @@
   </joint>
 </xacro:macro>
-<xacro:macro name="transmission" params="name joint_name actuator_name">
-  <transmission name="${name}">
-    <type>transmission_interface/SimpleTransmission</type>
-    <joint name="${joint_name}">
-      <hardwareInterface>hardware_interface/PositionJointInterface</hardwareInterface>
-    </joint>
-    <actuator name="${actuator_name}">
-      <hardwareInterface>hardware_interface/PositionJointInterface</hardwareInterface>
-      <mechanicalReduction>1</mechanicalReduction>
-    </actuator>
-  </transmission>
-</xacro:macro>
-<xacro:macro name="transmission_effort" params="name joint_name actuator_name">
-  <transmission name="${name}">
-    <type>transmission_interface/SimpleTransmission</type>
-    <joint name="${joint_name}">
-      <hardwareInterface>hardware_interface/EffortJointInterface</hardwareInterface>
-    </joint>
-    <actuator name="${actuator_name}">
-      <hardwareInterface>hardware_interface/EffortJointInterface</hardwareInterface>
-      <mechanicalReduction>1</mechanicalReduction>
-    </actuator>
-  </transmission>
+<xacro:macro name="arctos_control" params="name limit_u limit_l">
+  <joint name="${name}">
+    <command_interface name="position">
+          <param name="min">${limit_l}</param>
+          <param name="max">${limit_u}</param>
+    </command_interface>
+    <state_interface name="position"/>
+    <state_interface name="velocity"/>
+  </joint>
 </xacro:macro>
 </robot>

File: arctos_moveit/config/arctos.urdf.xacro (robot description, xacro)
@@ -3,5 +3,5 @@
     <xacro:arg name="initial_positions_file" default="initial_positions.yaml" />
     <!-- Import arctos urdf file -->
-    <xacro:include filename="$(find arctos_description)/urdf/arctos.xacro" />
+    <xacro:include filename="$(find arctos)/urdf/arctos.urdf.xacro" />
     <!-- Import control_xacro -->
     <xacro:include filename="arctos.ros2_control.xacro" />
